File: Hardware/Hardware.sch (KiCad schematic (older format))
At the start: 30 parts, among them P1 CONN_01X01, P2 CONN_01X01, P3 CONN_01X01, P4 CONN_01X01, U1 APE8865N-33-HF-3, U2 STM32F103RCT6, U3 MPU6050, Y1 8MHz

Commit message: doc: 4 layer PCB
Parts:
- added P5, P6, P7, P8: CONN_01X01, symbol CONN_01X01
Connections:
- net BLDC1: now reaches U2.22 (PA6/SPI1_MISO/TIM3_CH1)
- net BLDC1: now also P5.1 (P1)
- net BLDC2: now reaches U2.23 (PA7/SPI1_MOSI/TIM3_CH2)
- net BLDC2: now also P6.1 (P1)
- net BLDC3: now reaches U2.26 (PB0/ADC8/TIM3_CH3)
- net BLDC3: now also P7.1 (P1)
- net BLDC4: now reaches U2.27 (PB1/ADC9/TIM3_CH4)
- net BLDC4: now also P8.1 (P1)
- no-connect marks 51 -> 47
Changed lines of the file:
@@
 $EndComp
 $Comp
-L +3.3V #PWR01
+L +3.3V #PWR1
 U 1 1 5804A9FA
 P 1000 700
-F 0 "#PWR01" H 1000 550 50  0001 C CNN
+F 0 "#PWR1" H 1000 550 50  0001 C CNN
 F 1 "+3.3V" H 1000 840 50  0000 C CNN
 F 2 "" H 1000 700 50  0000 C CNN
@@
 $EndComp
 $Comp
-L GND #PWR02
+L GND #PWR5
 U 1 1 5804AA12
 P 1850 1400
-F 0 "#PWR02" H 1850 1150 50  0001 C CNN
+F 0 "#PWR5" H 1850 1150 50  0001 C CNN
 F 1 "GND" H 1850 1250 50  0000 C CNN
 F 2 "" H 1850 1400 50  0000 C CNN
@@
 $EndComp
 $Comp
-L GND #PWR03
+L GND #PWR4
 U 1 1 5804AA2A
 P 3900 850
-F 0 "#PWR03" H 3900 600 50  0001 C CNN
+F 0 "#PWR4" H 3900 600 50  0001 C CNN
 F 1 "GND" H 3900 700 50  0000 C CNN
 F 2 "" H 3900 850 50  0000 C CNN
@@
 $EndComp
 $Comp
-L +3.3V #PWR04
+L +3.3V #PWR3
 U 1 1 5804AA42
 P 3500 800
-F 0 "#PWR04" H 3500 650 50  0001 C CNN
+F 0 "#PWR3" H 3500 650 50  0001 C CNN
 F 1 "+3.3V" H 3500 940 50  0000 C CNN
 F 2 "" H 3500 800 50  0000 C CNN
@@
 $EndComp
 $Comp
-L PWR_FLAG #FLG05
+L PWR_FLAG #FLG1
 U 1 1 5804AA5A
 P 3500 800
-F 0 "#FLG05" H 3500 895 50  0001 C CNN
+F 0 "#FLG1" H 3500 895 50  0001 C CNN
 F 1 "PWR_FLAG" H 3500 980 50  0000 C CNN
 F 2 "" H 3500 800 50  0000 C CNN
@@
 $EndComp
 $Comp
-L PWR_FLAG #FLG06
+L PWR_FLAG #FLG2
 U 1 1 5804AA72
 P 3900 850
-F 0 "#FLG06" H 3900 945 50  0001 C CNN
+F 0 "#FLG2" H 3900 945 50  0001 C CNN
 F 1 "PWR_FLAG" H 3900 1030 50  0000 C CNN
 F 2 "" H 3900 850 50  0000 C CNN
@@
 $EndComp
 $Comp
-L GND #PWR07
+L GND #PWR8
 U 1 1 5804C0FA
 P 1100 2800
-F 0 "#PWR07" H 1100 2550 50  0001 C CNN
+F 0 "#PWR8" H 1100 2550 50  0001 C CNN
 F 1 "GND" H 1100 2650 50  0000 C CNN
 F 2 "" H 1100 2800 50  0000 C CNN
@@
 RESET
 $Comp
-L GND #PWR08
+L GND #PWR6
 U 1 1 5804C5B4
 P 1550 2000
-F 0 "#PWR08" H 1550 1750 50  0001 C CNN
+F 0 "#PWR6" H 1550 1750 50  0001 C CNN
 F 1 "GND" H 1550 1850 50  0000 C CNN
 F 2 "" H 1550 2000 50  0000 C CNN
@@
 $EndComp
 $Comp
-L GND #PWR09
+L GND #PWR2
 U 1 1 5804E93B
 P 5150 700
-F 0 "#PWR09" H 5150 450 50  0001 C CNN
+F 0 "#PWR2" H 5150 450 50  0001 C CNN
 F 1 "GND" H 5150 550 50  0000 C CNN
 F 2 "" H 5150 700 50  0000 C CNN
@@
 $EndComp
 $Comp
-L GND #PWR010
+L GND #PWR13
 U 1 1 5804F1CF
 P 950 6700
-F 0 "#PWR010" H 950 6450 50  0001 C CNN
+F 0 "#PWR13" H 950 6450 50  0001 C CNN
 F 1 "GND" H 950 6550 50  0000 C CNN
 F 2 "" H 950 6700 50  0000 C CNN
@@
 3V3
 $Comp
-L GND #PWR011
+L GND #PWR14
 U 1 1 5804F979
 P 950 7200
-F 0 "#PWR011" H 950 6950 50  0001 C CNN
+F 0 "#PWR14" H 950 6950 50  0001 C CNN
 F 1 "GND" H 950 7050 50  0000 C CNN
 F 2 "" H 950 7200 50  0000 C CNN
@@
 $EndComp
 $Comp
-L GND #PWR012
+L GND #PWR15
 U 1 1 58050959
 P 3100 7300
-F 0 "#PWR012" H 3100 7050 50  0001 C CNN
+F 0 "#PWR15" H 3100 7050 50  0001 C CNN
 F 1 "GND" H 3100 7150 50  0000 C CNN
 F 2 "" H 3100 7300 50  0000 C CNN
@@
 3V3
 $Comp
-L GND #PWR013
+L GND #PWR12
 U 1 1 58F83CEA
 P 7050 4950
-F 0 "#PWR013" H 7050 4700 50  0001 C CNN
+F 0 "#PWR12" H 7050 4700 50  0001 C CNN
 F 1 "GND" H 7050 4800 50  0000 C CNN
 F 2 "" H 7050 4950 50  0000 C CNN
@@
 3V3
 $Comp
-L GND #PWR014
+L GND #PWR10
 U 1 1 58F84302
 P 7050 3650
-F 0 "#PWR014" H 7050 3400 50  0001 C CNN
+F 0 "#PWR10" H 7050 3400 50  0001 C CNN
 F 1 "GND" H 7050 3500 50  0000 C CNN
 F 2 "" H 7050 3650 50  0000 C CNN
@@
 3V3
 $Comp
-L GND #PWR015
+L GND #PWR9
 U 1 1 58F84436
 P 7050 2950
-F 0 "#PWR015" H 7050 2700 50  0001 C CNN
+F 0 "#PWR9" H 7050 2700 50  0001 C CNN
 F 1 "GND" H 7050 2800 50  0000 C CNN
 F 2 "" H 7050 2950 50  0000 C CNN
@@
 3V3
 $Comp
-L GND #PWR016
+L GND #PWR7
 U 1 1 58F8457A
 P 10750 2150
-F 0 "#PWR016" H 10750 1900 50  0001 C CNN
+F 0 "#PWR7" H 10750 1900 50  0001 C CNN
 F 1 "GND" H 10750 2000 50  0000 C CNN
 F 2 "" H 10750 2150 50  0000 C CNN
@@
 3V3
 $Comp
-L GND #PWR017
+L GND #PWR11
 U 1 1 58F8482A
 P 10750 3850
-F 0 "#PWR017" H 10750 3600 50  0001 C CNN
+F 0 "#PWR11" H 10750 3600 50  0001 C CNN
 F 1 "GND" H 10750 3700 50  0000 C CNN
 F 2 "" H 10750 3850 50  0000 C CNN
@@
 NoConn ~ 7700 3450
 NoConn ~ 7700 3650
-NoConn ~ 7700 3950
 NoConn ~ 7700 4050
-NoConn ~ 7700 4150
-NoConn ~ 7700 4250
 NoConn ~ 7700 4350
 NoConn ~ 7700 4450
-NoConn ~ 7700 4550
-NoConn ~ 7700 4650
 NoConn ~ 7700 4850
 NoConn ~ 7700 4950
@@
 NoConn ~ 10100 2250
 NoConn ~ 10100 2150
+$Comp
+L CONN_01X01 P5
+U 1 1 58F878C0
+P 6400 5850
+F 0 "P5" H 6400 5950 50  0000 C CNN
+F 1 "CONN_01X01" V 6500 5850 50  0000 C CNN
+F 2 "" H 6400 5850 50  0000 C CNN
+F 3 "" H 6400 5850 50  0000 C CNN
+	1    6400 5850
+	1    0    0    -1
+$EndComp
+$Comp
+L CONN_01X01 P6
+U 1 1 58F87930
+P 6400 6350
+F 0 "P6" H 6400 6450 50  0000 C CNN
+F 1 "CONN_01X01" V 6500 6350 50  0000 C CNN
+F 2 "" H 6400 6350 50  0000 C CNN
+F 3 "" H 6400 6350 50  0000 C CNN
+	1    6400 6350
+	1    0    0    -1
+$EndComp
+$Comp
+L CONN_01X01 P7
+U 1 1 58F87991
+P 6400 6850
+F 0 "P7" H 6400 6950 50  0000 C CNN
+F 1 "CONN_01X01" V 6500 6850 50  0000 C CNN
+F 2 "" H 6400 6850 50  0000 C CNN
+F 3 "" H 6400 6850 50  0000 C CNN
+	1    6400 6850
+	1    0    0    -1
+$EndComp
+$Comp
+L CONN_01X01 P8
+U 1 1 58F879E8
+P 6400 7350
+F 0 "P8" H 6400 7450 50  0000 C CNN
+F 1 "CONN_01X01" V 6500 7350 50  0000 C CNN
+F 2 "" H 6400 7350 50  0000 C CNN
+F 3 "" H 6400 7350 50  0000 C CNN
+	1    6400 7350
+	1    0    0    -1
+$EndComp
+NoConn ~ 7700 3950
+Text GLabel 7700 4150 0    60   Input ~ 0
+BLDC1
+Text GLabel 7700 4250 0    60   Input ~ 0
+BLDC2
+Text GLabel 7700 4550 0    60   Input ~ 0
+BLDC3
+Text GLabel 7700 4650 0    60   Input ~ 0
+BLDC4
+Text GLabel 6200 5850 0    60   Input ~ 0
+BLDC1
+Text GLabel 6200 6350 0    60   Input ~ 0
+BLDC2
+Text GLabel 6200 6850 0    60   Input ~ 0
+BLDC3
+Text GLabel 6200 7350 0    60   Input ~ 0
+BLDC4
 $EndSCHEMATC
