File: Platform/platform.sch (KiCad schematic (older format))
At the start: 18 parts, among them P1 VCC, P10 -, P11 CH3, P12 CH3, P13 RX, P14 RX, P15 CH4, P16 CH4, P17 TX, P18 TX, P2 GND, P3 CH1, P4 CH1, P5 +, P6 +, P7 CH2, P8 CH2, P9 -

Commit message: doc: (platform)
Parts:
- added P10, P7, P8, P9: GND, symbol CONN_01X01
- added P3, P4, P5, P6: VCC, symbol CONN_01X01
- renumbered P3 to P11, P4 to P12, P5 to P13, P6 to P14, P7 to P15, P8 to P16, P9 to P17, P10 to P18, P11 to P19, P12 to P20, P13 to P21, P14 to P22, P15 to P23, P16 to P24, P17 to P25, P18 to P26
Connections:
- net +5V: now also P3.1 (P1), P4.1 (P1), P5.1 (P1), P6.1 (P1)
- net GND: now also P10.1 (P1), P7.1 (P1), P8.1 (P1), P9.1 (P1)
Other:
- note added: "PWM\n"
- note added: "Power Hub\n"
- note added: "Power Input\n"
- note added: "UART\n"
- moved on the sheet: P1, P11, P12, P13, P14, P15, P16, P17, P18, P19, P2, P20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
